File: KiCad/LPFilter_100kHz_Elliptical_v0.1/LPFilter_100kHz_Elliptical_v0.1.kicad_sch (KiCad schematic)
At the start: 15 parts, among them J1 IN, J2 OUT

Commit message: Commit Fixes
Parts:
- removed G1: IAMSnanofiber, IAMS:IAMSnanofiber, symbol IAMS:IAMSnanofiber
- removed G2: IAMS, IAMS:IAMS, symbol IAMS:IAMS
- removed G3: IAMSYb, IAMS:IAMSYb, symbol IAMS:IAMSYb
