File: KiCad/LPFilter_200kHz_Elliptical_v0.1/LPFilter_200kHz_Elliptical_v0.1.kicad_pcb (KiCad board)
At the start: 4 copper layers, 77 x 21.5 mm, 16 parts, among them J1 IN, J2 OUT

Commit message: Commit Fixes
Parts:
- removed G1: IAMSnanofiber, IAMS:IAMSnanofiber
- removed G2: IAMS, IAMS:IAMS
- removed G3: IAMSYb, IAMS:IAMSYb
